Commit message: Adicionado novo codigo

File: robot_one_description/urdf/robot_one.xacro (robot description, xacro)
@@ -26,5 +26,4 @@
       </collision>
   </link>
-  <!-- Roda Castor Frontal -->
   <link name="front_caster">
     <inertial>
@@ -38,5 +37,5 @@
         <origin xyz="0 0 0" rpy="-1.5707 0 1.5707" />
         <geometry>
-          <mesh filename="package://abrobot_description/meshes/castor.dae"/>
+          <mesh filename="package://robot_one_description/meshes/castor.dae"/>
         </geometry>
         <material name ="light_grey">
@@ -47,5 +46,5 @@
         <origin xyz="0 0 0" rpy="-1.5707 0 1.5707" />
         <geometry>
-          <cylinder length="0.0605" radius="0.097"/>
+          <mesh filename="package://robot_one_description/meshes/castor.dae"/>
         </geometry>
       </collision>
@@ -67,5 +66,5 @@
         <origin xyz="0 0 0" rpy="-1.5707 0 1.5707" />
         <geometry>
-          <mesh filename="package://abrobot_description/meshes/castor.dae"/>
+          <mesh filename="package://robot_one_description/meshes/castor.dae"/>
         </geometry>
         <material name ="light_grey">
@@ -76,5 +75,5 @@
         <origin xyz="0 0 0" rpy="-1.5707 0 1.5707" />
         <geometry>
-          <cylinder length="0.0605" radius="0.097"/>
+			<mesh filename="package://robot_one_description/meshes/castor.dae"/>
         </geometry>
       </collision>
@@ -85,4 +84,5 @@
     <child link="rear_caster" />
   </joint>
+  <!-- Roda Castor Frontal -->
   <link name="left_axle_link">
     <inertial>
@@ -108,5 +108,5 @@
   <joint name="left_axle_joint" type="fixed">
     <origin xyz="0 0.171475 0.017" rpy="0 0 0"/>
-    <parent link="battery_box"/>
+    <parent link="base_link"/>
     <child link="left_axle_link"/>
     <axis xyz="0 1 0"/>
@@ -135,5 +135,5 @@
   <joint name="right_axle_joint" type="fixed">
     <origin xyz="0 -0.171475 0.017" rpy="0 0 0"/>
-    <parent link="battery_box"/>
+    <parent link="base_link"/>
     <child link="right_axle_link"/>
     <axis xyz="0 1 0"/>
@@ -147,5 +147,5 @@
       </inertial>
       <visual>
-        <origin xyz="0 0 0" rpy="0 1.5707 1.5707" />
+        <origin xyz="0 0 -0.040" rpy="0 1.5707 1.5707" />
         <geometry>
           <cylinder radius="0.0762" length = "0.03175"/>
@@ -154,5 +154,5 @@
       </visual>
       <collision>
-        <origin xyz="0 0 0" rpy="0 1.5707 1.5707" />
+        <origin xyz="0 0 -0.040" rpy="0 1.5707 1.5707" />
         <geometry>
           <cylinder radius="0.076" length = "0.03175"/>
@@ -187,6 +187,4 @@
       </collision>
   </link>
-  <!-- Fixed because we never rotate it anyway, it is just for show -->
-  <!-- NOTE This may prevent gazebo from working with this model -->
   <joint name="right_wheel_joint" type="continuous">
     <origin xyz="0 -0.01905 0" rpy="0 0 0"/>

Commit message: Inicio - Programa Funcional

File: robot_one_description/urdf/robot_one.xacro (robot description, xacro)
@@ -4,4 +4,7 @@
   <xacro:include filename="$(find robot_one_description)/urdf/materials.xacro" />
   <!-- <xacro:include filename="$(find abrobot_description)/urdf/macros.xacro"/> -->
+  <xacro:property name="DIAMETRO_ROBO" value="0.60"/>
+  <xacro:property name="EIXO_ROBO" value="0.05"/>
+  <xacro:property name="M_PI" value="3.1415926535897931" />
   <!-- Base Robotic -->
   <link name="base_link">
@@ -15,5 +18,5 @@
         <origin xyz="0 0 0" rpy="0 0 0" />
         <geometry>
-          <cylinder length="0.0095" radius="0.2245"/>
+          <cylinder length="0.0095" radius="${DIAMETRO_ROBO/2}"/>
         </geometry>
         <material name ="White" />
@@ -22,8 +25,9 @@
         <origin xyz="0 0 0" rpy="0 0 0" />
         <geometry>
-          <cylinder length="0.0095" radius="0.2245"/>
-        </geometry>
-      </collision>
-  </link>
+          <cylinder length="0.0095" radius="${DIAMETRO_ROBO/2}"/>
+        </geometry>
+      </collision>
+  </link>
+  <!-- Roda Castor Frontal -->
   <link name="front_caster">
     <inertial>
@@ -55,4 +59,5 @@
     <child link="front_caster" />
   </joint>
+  <!-- Roda Castor Traseira -->
   <link name="rear_caster">
     <inertial>
@@ -75,5 +80,5 @@
         <origin xyz="0 0 0" rpy="-1.5707 0 1.5707" />
         <geometry>
-			<mesh filename="package://robot_one_description/meshes/castor.dae"/>
+          <mesh filename="package://robot_one_description/meshes/castor.dae"/>
         </geometry>
       </collision>
@@ -84,5 +89,5 @@
     <child link="rear_caster" />
   </joint>
-  <!-- Roda Castor Frontal -->
+  <!-- Eixo Roda Esquerda -->
   <link name="left_axle_link">
     <inertial>
@@ -95,5 +100,5 @@
         <origin xyz="0 0 0" rpy="0 1.5707 1.5707" />
         <geometry>
-          <cylinder radius="0.00635" length = "0.00635"/>
+          <cylinder radius="0.00635" length = "${EIXO_ROBO}"/>
         </geometry>
         <material name ="light_grey" />
@@ -102,14 +107,15 @@
         <origin xyz="0 0 0" rpy="0 1.5707 1.5707" />
         <geometry>
-          <cylinder radius="0.00635" length = "0.00635"/>
+          <cylinder radius="0.00635" length = "${EIXO_ROBO}"/>
         </geometry>
       </collision>
   </link>
   <joint name="left_axle_joint" type="fixed">
-    <origin xyz="0 0.171475 0.017" rpy="0 0 0"/>
+    <origin xyz="0 -${DIAMETRO_ROBO/2} 0" rpy="0 0 0"/>
     <parent link="base_link"/>
     <child link="left_axle_link"/>
     <axis xyz="0 1 0"/>
   </joint>
+  <!-- Eixo Roda Direita -->
   <link name="right_axle_link">
     <inertial>
@@ -120,32 +126,32 @@
       </inertial>
       <visual>
-        <origin xyz="0 0 0" rpy="0 1.5707 1.5707" />
-        <geometry>
-          <cylinder radius="0.00635" length = "0.00635"/>
+        <origin xyz="0 0 0" rpy="0 ${M_PI/2} ${M_PI/2}" />
+        <geometry>
+          <cylinder radius="0.00635" length = "${EIXO_ROBO}"/>
         </geometry>
         <material name ="light_grey" />
       </visual>
       <collision>
-        <origin xyz="0 0 0" rpy="0 1.5707 1.5707" />
-        <geometry>
-          <cylinder radius="0.00635" length = "0.00635"/>
+        <origin xyz="0 0 0" rpy="0 ${M_PI/2} ${M_PI/2}" />
+        <geometry>
+          <cylinder radius="0.00635" length = "${EIXO_ROBO}"/>
         </geometry>
       </collision>
   </link>
   <joint name="right_axle_joint" type="fixed">
-    <origin xyz="0 -0.171475 0.017" rpy="0 0 0"/>
+    <origin xyz="0 ${DIAMETRO_ROBO/2} 0" rpy="0 0 0"/>
     <parent link="base_link"/>
     <child link="right_axle_link"/>
     <axis xyz="0 1 0"/>
-  </joint>
-  <link name="left_wheel_link">
-    <inertial>
-      <origin xyz="0 0 0"/>
-      <mass value="0.01" />
-      <inertia ixx="0.001" ixy="0.0" ixz="0.0"
-        iyy="0.001" iyz="0.0" izz="0.001" />
-      </inertial>
-      <visual>
-        <origin xyz="0 0 -0.040" rpy="0 1.5707 1.5707" />
+  </joint> -->
+  <!-- <link name="left_wheel_link">
+    <inertial>
+      <origin xyz="0 0 0"/>
+      <mass value="0.01" />
+      <inertia ixx="0.001" ixy="0.0" ixz="0.0"
+        iyy="0.001" iyz="0.0" izz="0.001" />
+      </inertial>
+      <visual>
+        <origin xyz="0 0 0" rpy="0 1.5707 1.5707" />
         <geometry>
           <cylinder radius="0.0762" length = "0.03175"/>
@@ -154,5 +160,5 @@
       </visual>
       <collision>
-        <origin xyz="0 0 -0.040" rpy="0 1.5707 1.5707" />
+        <origin xyz="0 0 0" rpy="0 1.5707 1.5707" />
         <geometry>
           <cylinder radius="0.076" length = "0.03175"/>
@@ -165,6 +171,6 @@
     <child link="left_wheel_link"/>
     <axis xyz="0 1 0"/>
-  </joint>
-  <link name="right_wheel_link">
+  </joint> -->
+  <!-- <link name="right_wheel_link">
     <inertial>
       <origin xyz="0 0 0"/>
@@ -186,10 +192,12 @@
         </geometry>
       </collision>
-  </link>
-  <joint name="right_wheel_joint" type="continuous">
+  </link> -->
+  <!-- Fixed because we never rotate it anyway, it is just for show -->
+  <!-- NOTE This may prevent gazebo from working with this model -->
+<!--   <joint name="right_wheel_joint" type="continuous">
     <origin xyz="0 -0.01905 0" rpy="0 0 0"/>
     <parent link="right_axle_link"/>
     <child link="right_wheel_link"/>
     <axis xyz="0 1 0"/>
-  </joint>
+  </joint> -->
 </robot>

Commit message: Atualizado

File: robot_one_description/urdf/robot_one.xacro (robot description, xacro)
@@ -3,5 +3,7 @@
   <xacro:include filename="$(find robot_one_description)/urdf/robot_one.gazebo" />
   <xacro:include filename="$(find robot_one_description)/urdf/materials.xacro" />
-  <!-- <xacro:include filename="$(find abrobot_description)/urdf/macros.xacro"/> -->
+  <xacro:property name="D_ROBO" value="0.5" />
+  <xacro:property name="EIXO_ROBO" value="0.00635" />
+  <xacro:property name="PI" value="3.1415926535897931" />
   <!-- Base Robotic -->
   <link name="base_link">
@@ -15,5 +17,5 @@
         <origin xyz="0 0 0" rpy="0 0 0" />
         <geometry>
-          <cylinder length="0.0095" radius="0.2245"/>
+          <cylinder length="0.0095" radius="${D_ROBO/2}"/>
         </geometry>
         <material name ="White" />
@@ -22,8 +24,9 @@
         <origin xyz="0 0 0" rpy="0 0 0" />
         <geometry>
-          <cylinder length="0.0095" radius="0.2245"/>
+          <cylinder length="0.0095" radius="${D_ROBO/2}"/>
         </geometry>
       </collision>
   </link>
+  <!-- Caster Whells -->
   <link name="front_caster">
     <inertial>
@@ -75,5 +78,5 @@
         <origin xyz="0 0 0" rpy="-1.5707 0 1.5707" />
         <geometry>
-			<mesh filename="package://robot_one_description/meshes/castor.dae"/>
+      <mesh filename="package://robot_one_description/meshes/castor.dae"/>
         </geometry>
       </collision>
@@ -84,5 +87,5 @@
     <child link="rear_caster" />
   </joint>
-  <!-- Roda Castor Frontal -->
+  <!-- Axles -->
   <link name="left_axle_link">
     <inertial>
@@ -93,19 +96,19 @@
       </inertial>
       <visual>
-        <origin xyz="0 0 0" rpy="0 1.5707 1.5707" />
+        <origin xyz="0 0 0" rpy="0 ${PI/2} ${PI/2}" />
         <geometry>
-          <cylinder radius="0.00635" length = "0.00635"/>
+          <cylinder radius="${EIXO_ROBO}" length = "${EIXO_ROBO}"/>
         </geometry>
         <material name ="light_grey" />
       </visual>
       <collision>
-        <origin xyz="0 0 0" rpy="0 1.5707 1.5707" />
+        <origin xyz="0 0 0" rpy="0 ${PI/2} ${PI/2}" />
         <geometry>
-          <cylinder radius="0.00635" length = "0.00635"/>
+          <cylinder radius="${EIXO_ROBO}" length = "${EIXO_ROBO}"/>
         </geometry>
       </collision>
   </link>
   <joint name="left_axle_joint" type="fixed">
-    <origin xyz="0 0.171475 0.017" rpy="0 0 0"/>
+    <origin xyz="0 ${D_ROBO/2 + EIXO_ROBO} 0" rpy="0 0 0"/>
     <parent link="base_link"/>
     <child link="left_axle_link"/>
@@ -120,23 +123,24 @@
       </inertial>
       <visual>
-        <origin xyz="0 0 0" rpy="0 1.5707 1.5707" />
+        <origin xyz="0 0 0" rpy="0 ${PI/2} ${PI/2}" />
         <geometry>
-          <cylinder radius="0.00635" length = "0.00635"/>
+          <cylinder radius="${EIXO_ROBO}" length = "${EIXO_ROBO}"/>
         </geometry>
         <material name ="light_grey" />
       </visual>
       <collision>
-        <origin xyz="0 0 0" rpy="0 1.5707 1.5707" />
+        <origin xyz="0 0 0" rpy="0 ${PI/2} ${PI/2}" />
         <geometry>
-          <cylinder radius="0.00635" length = "0.00635"/>
+          <cylinder radius="${EIXO_ROBO}" length = "${EIXO_ROBO}"/>
         </geometry>
       </collision>
   </link>
   <joint name="right_axle_joint" type="fixed">
-    <origin xyz="0 -0.171475 0.017" rpy="0 0 0"/>
+    <origin xyz="0 -${D_ROBO/2 + EIXO_ROBO} 0" rpy="0 0 0"/>
     <parent link="base_link"/>
     <child link="right_axle_link"/>
     <axis xyz="0 1 0"/>
   </joint>
+  <!-- Wheels -->
   <link name="left_wheel_link">
     <inertial>
@@ -147,5 +151,5 @@
       </inertial>
       <visual>
-        <origin xyz="0 0 -0.040" rpy="0 1.5707 1.5707" />
+        <origin xyz="0 0 0" rpy="0 1.5707 1.5707" />
         <geometry>
           <cylinder radius="0.0762" length = "0.03175"/>
@@ -154,5 +158,5 @@
       </visual>
       <collision>
-        <origin xyz="0 0 -0.040" rpy="0 1.5707 1.5707" />
+        <origin xyz="0 0 0" rpy="0 1.5707 1.5707" />
         <geometry>
           <cylinder radius="0.076" length = "0.03175"/>

Commit message: add teleop

File: robot_one_description/urdf/robot_one.xacro (robot description, xacro)
@@ -6,4 +6,5 @@
   <xacro:property name="EIXO_ROBO" value="0.00635" />
   <xacro:property name="PI" value="3.1415926535897931" />
+  <xacro:property name="D_RODA" value="0.104" />
   <!-- Base Robotic -->
   <link name="base_link">
@@ -153,5 +154,5 @@
         <origin xyz="0 0 0" rpy="0 1.5707 1.5707" />
         <geometry>
-          <cylinder radius="0.0762" length = "0.03175"/>
+          <cylinder radius="${D_RODA}" length = "0.03175"/>
         </geometry>
         <material name ="black" />
@@ -160,5 +161,5 @@
         <origin xyz="0 0 0" rpy="0 1.5707 1.5707" />
         <geometry>
-          <cylinder radius="0.076" length = "0.03175"/>
+          <cylinder radius="${D_RODA}" length = "0.03175"/>
         </geometry>
       </collision>
@@ -180,5 +181,5 @@
         <origin xyz="0 0 0" rpy="0 1.5707 1.5707" />
         <geometry>
-          <cylinder radius="0.0762" length = "0.03175"/>
+          <cylinder radius="${D_RODA}" length = "0.03175"/>
         </geometry>
         <material name ="black" />
@@ -187,5 +188,5 @@
         <origin xyz="0 0 0" rpy="0 1.5707 1.5707" />
         <geometry>
-          <cylinder radius="0.076" length = "0.03175"/>
+          <cylinder radius="${D_RODA}" length = "0.03175"/>
         </geometry>
       </collision>

Commit message: add LIDAR and Real Sense

File: robot_one_description/urdf/robot_one.xacro (robot description, xacro)
@@ -6,5 +6,5 @@
   <xacro:property name="EIXO_ROBO" value="0.00635" />
   <xacro:property name="PI" value="3.1415926535897931" />
-  <xacro:property name="D_RODA" value="0.104" />
+  <xacro:property name="D_RODA" value="0.105" />
   <!-- Base Robotic -->
   <link name="base_link">
@@ -198,3 +198,81 @@
     <axis xyz="0 1 0"/>
   </joint>
+  <!-- LIDAR -->
+<link name="base_laser">
+    <collision>
+      <origin xyz="0 0 0" rpy="0 0 0"/>
+      <geometry>
+        <box size="0.1 0.1 0.1"/>
+      </geometry>
+    </collision>
+    <visual>
+      <origin xyz="0 0 -0.03" rpy="0 0 0"/>
+      <geometry>
+        <mesh filename="package://robot_one_description/meshes/rplidar.stl" scale="0.01 0.01 0.01" />
+      </geometry>
+    </visual>
+    <inertial>
+      <mass value="1e-5" />
+      <origin xyz="0 0 0" rpy="0 0 0"/>
+      <inertia ixx="1e-6" ixy="0" ixz="0" iyy="1e-6" iyz="0" izz="1e-6" />
+    </inertial>
+  </link>
+  <joint name="laser_joint" type="fixed">
+    <axis xyz="0 0 0" />
+    <origin xyz="0 0 0.1" rpy="0 0 0"/>
+    <parent link="base_link"/>
+    <child link="base_laser"/>
+  </joint>
+  <!-- Real Sense -->
+  <!-- LIDAR -->
+<link name="Front_Real_Sense">
+    <collision>
+      <origin xyz="0 0 0" rpy="0 0 0"/>
+      <geometry>
+        <mesh filename="package://robot_one_description/meshes/IntelRealsense_D435_Multibody.stl" scale="0.01 0.01 0.01" />
+      </geometry>
+    </collision>
+    <visual>
+      <origin xyz="0 0 0" rpy="0 0 0"/>
+      <geometry>
+        <mesh filename="package://robot_one_description/meshes/IntelRealsense_D435_Multibody.stl" scale="0.01 0.01 0.01" />
+      </geometry>
+    </visual>
+    <inertial>
+      <mass value="1e-5" />
+      <origin xyz="0 0 0" rpy="0 0 0"/>
+      <inertia ixx="1e-6" ixy="0" ixz="0" iyy="1e-6" iyz="0" izz="1e-6" />
+    </inertial>
+  </link>
+  <joint name="Front_Real_Sense_joint" type="fixed">
+    <axis xyz="0 0 0" />
+    <origin xyz="0.2 0 0.07" rpy="-${PI/2} 0 -${PI/2}"/>
+    <parent link="base_link"/>
+    <child link="Front_Real_Sense"/>
+  </joint>
+<link name="Rear_Real_Sense">
+    <collision>
+      <origin xyz="0 0 0" rpy="0 0 0"/>
+      <geometry>
+        <mesh filename="package://robot_one_description/meshes/IntelRealsense_D435_Multibody.stl" scale="0.01 0.01 0.01" />
+      </geometry>
+    </collision>
+    <visual>
+      <origin xyz="0 0 0" rpy="0 0 0"/>
+      <geometry>
+        <mesh filename="package://robot_one_description/meshes/IntelRealsense_D435_Multibody.stl" scale="0.01 0.01 0.01" />
+      </geometry>
+    </visual>
+    <inertial>
+      <mass value="1e-5" />
+      <origin xyz="0 0 0" rpy="0 0 0"/>
+      <inertia ixx="1e-6" ixy="0" ixz="0" iyy="1e-6" iyz="0" izz="1e-6" />
+    </inertial>
+  </link>
+  <joint name="Rear_Real_Sense_joint" type="fixed">
+    <axis xyz="0 0 0" />
+    <origin xyz="-0.2 0 0.07" rpy="-${PI/2} 0 ${PI/2}"/>
+    <parent link="base_link"/>
+    <child link="Rear_Real_Sense"/>
+  </joint>
 </robot>

Commit message: Add lidar

File: robot_one_description/urdf/robot_one.xacro (robot description, xacro)
@@ -220,10 +220,9 @@
   <joint name="laser_joint" type="fixed">
     <axis xyz="0 0 0" />
-    <origin xyz="0 0 0.1" rpy="0 0 0"/>
+    <origin xyz="0 0 0.2" rpy="0 0 0"/>
     <parent link="base_link"/>
     <child link="base_laser"/>
   </joint>
   <!-- Real Sense -->
-  <!-- LIDAR -->
 <link name="Front_Real_Sense">
     <collision>

Commit message: Add Camera Real Sense

File: robot_one_description/urdf/robot_one.xacro (robot description, xacro)
@@ -225,5 +225,5 @@
   </joint>
   <!-- Real Sense -->
-<link name="Front_Real_Sense">
+<link name="Front_Camera">
     <collision>
       <origin xyz="0 0 0" rpy="0 0 0"/>
@@ -244,11 +244,11 @@
     </inertial>
   </link>
-  <joint name="Front_Real_Sense_joint" type="fixed">
+  <joint name="Front_Camera_joint" type="fixed">
     <axis xyz="0 0 0" />
     <origin xyz="0.2 0 0.07" rpy="-${PI/2} 0 -${PI/2}"/>
     <parent link="base_link"/>
-    <child link="Front_Real_Sense"/>
-  </joint>
-<link name="Rear_Real_Sense">
+    <child link="Front_Camera"/>
+  </joint>
+<link name="Rear_Camera">
     <collision>
       <origin xyz="0 0 0" rpy="0 0 0"/>
@@ -269,9 +269,9 @@
     </inertial>
   </link>
-  <joint name="Rear_Real_Sense_joint" type="fixed">
+  <joint name="Rear_Camera_joint" type="fixed">
     <axis xyz="0 0 0" />
     <origin xyz="-0.2 0 0.07" rpy="-${PI/2} 0 ${PI/2}"/>
     <parent link="base_link"/>
-    <child link="Rear_Real_Sense"/>
+    <child link="Rear_Camera"/>
   </joint>
 </robot>

Commit message: Add README.md

File: robot_one_description/urdf/robot_one.xacro (robot description, xacro)
@@ -39,5 +39,5 @@
     </inertial>
       <visual>
-        <origin xyz="0 0 0" rpy="-1.5707 0 1.5707" />
+        <origin xyz="0 0 0" rpy="-${PI/2} 0 ${PI/2}" />
         <geometry>
           <mesh filename="package://robot_one_description/meshes/castor.dae"/>
@@ -48,5 +48,5 @@
       </visual>
       <collision>
-        <origin xyz="0 0 0" rpy="-1.5707 0 1.5707" />
+        <origin xyz="0 0 0" rpy="-${PI/2} 0 ${PI/2}" />
         <geometry>
           <mesh filename="package://robot_one_description/meshes/castor.dae"/>
@@ -68,5 +68,5 @@
       </inertial>
       <visual>
-        <origin xyz="0 0 0" rpy="-1.5707 0 1.5707" />
+        <origin xyz="0 0 0" rpy="-${PI/2} 0 ${PI/2}" />
         <geometry>
           <mesh filename="package://robot_one_description/meshes/castor.dae"/>
@@ -77,5 +77,5 @@
       </visual>
       <collision>
-        <origin xyz="0 0 0" rpy="-1.5707 0 1.5707" />
+        <origin xyz="0 0 0" rpy="-${PI/2} 0 ${PI/2}" />
         <geometry>
       <mesh filename="package://robot_one_description/meshes/castor.dae"/>
@@ -152,5 +152,5 @@
       </inertial>
       <visual>
-        <origin xyz="0 0 0" rpy="0 1.5707 1.5707" />
+        <origin xyz="0 0 0" rpy="0 ${PI/2} ${PI/2}" />
         <geometry>
           <cylinder radius="${D_RODA}" length = "0.03175"/>
@@ -159,5 +159,5 @@
       </visual>
       <collision>
-        <origin xyz="0 0 0" rpy="0 1.5707 1.5707" />
+        <origin xyz="0 0 0" rpy="0 ${PI/2} ${PI/2}" />
         <geometry>
           <cylinder radius="${D_RODA}" length = "0.03175"/>
@@ -179,5 +179,5 @@
       </inertial>
       <visual>
-        <origin xyz="0 0 0" rpy="0 1.5707 1.5707" />
+        <origin xyz="0 0 0" rpy="0 ${PI/2} ${PI/2}" />
         <geometry>
           <cylinder radius="${D_RODA}" length = "0.03175"/>
@@ -186,5 +186,5 @@
       </visual>
       <collision>
-        <origin xyz="0 0 0" rpy="0 1.5707 1.5707" />
+        <origin xyz="0 0 0" rpy="0 ${PI/2} ${PI/2}" />
         <geometry>
           <cylinder radius="${D_RODA}" length = "0.03175"/>

Commit message: Fixed

File: robot_one_description/urdf/robot_one.xacro (robot description, xacro)
@@ -203,5 +203,5 @@
       <origin xyz="0 0 0" rpy="0 0 0"/>
       <geometry>
-        <box size="0.1 0.1 0.1"/>
+         <mesh filename="package://robot_one_description/meshes/rplidar.stl" scale="0.01 0.01 0.01" />
       </geometry>
     </collision>
@@ -227,5 +227,5 @@
 <link name="Front_Camera">
     <collision>
-      <origin xyz="0 0 0" rpy="0 0 0"/>
+      <origin xyz="0 0 0" rpy="${PI/2} 0 ${PI/2}"/>
       <geometry>
         <mesh filename="package://robot_one_description/meshes/IntelRealsense_D435_Multibody.stl" scale="0.01 0.01 0.01" />
@@ -233,5 +233,5 @@
     </collision>
     <visual>
-      <origin xyz="0 0 0" rpy="0 0 0"/>
+      <origin xyz="0 0 0" rpy="${PI/2} 0 ${PI/2}"/>
       <geometry>
         <mesh filename="package://robot_one_description/meshes/IntelRealsense_D435_Multibody.stl" scale="0.01 0.01 0.01" />
@@ -240,11 +240,11 @@
     <inertial>
       <mass value="1e-5" />
-      <origin xyz="0 0 0" rpy="0 0 0"/>
+      <origin xyz="0 0 0" rpy="${PI/2} 0 ${PI/2}"/>
       <inertia ixx="1e-6" ixy="0" ixz="0" iyy="1e-6" iyz="0" izz="1e-6" />
     </inertial>
   </link>
   <joint name="Front_Camera_joint" type="fixed">
-    <axis xyz="0 0 0" />
-    <origin xyz="0.2 0 0.07" rpy="-${PI/2} 0 -${PI/2}"/>
+    <axis xyz="0 1 0" />
+    <origin xyz="0.1995 0 0.035" rpy="0 0 0"/>
     <parent link="base_link"/>
     <child link="Front_Camera"/>
@@ -252,5 +252,5 @@
 <link name="Rear_Camera">
     <collision>
-      <origin xyz="0 0 0" rpy="0 0 0"/>
+      <origin xyz="0 0 0" rpy="${PI/2} 0 ${PI/2}"/>
       <geometry>
         <mesh filename="package://robot_one_description/meshes/IntelRealsense_D435_Multibody.stl" scale="0.01 0.01 0.01" />
@@ -258,5 +258,5 @@
     </collision>
     <visual>
-      <origin xyz="0 0 0" rpy="0 0 0"/>
+      <origin xyz="0 0 0" rpy="${PI/2} 0 ${PI/2}"/>
       <geometry>
         <mesh filename="package://robot_one_description/meshes/IntelRealsense_D435_Multibody.stl" scale="0.01 0.01 0.01" />
@@ -265,11 +265,11 @@
     <inertial>
       <mass value="1e-5" />
-      <origin xyz="0 0 0" rpy="0 0 0"/>
+      <origin xyz="0 0 0" rpy="${PI/2} 0 ${PI/2}"/>
       <inertia ixx="1e-6" ixy="0" ixz="0" iyy="1e-6" iyz="0" izz="1e-6" />
     </inertial>
   </link>
   <joint name="Rear_Camera_joint" type="fixed">
-    <axis xyz="0 0 0" />
-    <origin xyz="-0.2 0 0.07" rpy="-${PI/2} 0 ${PI/2}"/>
+    <axis xyz="0 1 0" />
+    <origin xyz="-0.1995 0 0.035" rpy="0 0 ${PI}"/>
     <parent link="base_link"/>
     <child link="Rear_Camera"/>
