Commit message: Add all README

File: robot_one_description/urdf/robot_one.xacro (robot description, xacro)
@@ -20,5 +20,5 @@
           <cylinder length="0.0095" radius="${D_ROBO/2}"/>
         </geometry>
-        <material name ="White" />
+        <material name ="orange" />
       </visual>
       <collision>
@@ -156,5 +156,5 @@
           <cylinder radius="${D_RODA}" length = "0.03175"/>
         </geometry>
-        <material name ="black" />
+        <material name ="blue" />
       </visual>
       <collision>
@@ -183,5 +183,5 @@
           <cylinder radius="${D_RODA}" length = "0.03175"/>
         </geometry>
-        <material name ="black" />
+        <material name ="blue" />
       </visual>
       <collision>
@@ -211,4 +211,5 @@
         <mesh filename="package://robot_one_description/meshes/rplidar.stl" scale="0.01 0.01 0.01" />
       </geometry>
+      <material name ="blue" />
     </visual>
     <inertial>
@@ -237,4 +238,5 @@
         <mesh filename="package://robot_one_description/meshes/IntelRealsense_D435_Multibody.stl" scale="0.01 0.01 0.01" />
       </geometry>
+      <material name ="green" />
     </visual>
     <inertial>
@@ -262,4 +264,5 @@
         <mesh filename="package://robot_one_description/meshes/IntelRealsense_D435_Multibody.stl" scale="0.01 0.01 0.01" />
       </geometry>
+      <material name ="green" />
     </visual>
     <inertial>
